File: AVSwitch-Composite/AVSwitch-Composite.kicad_pcb (KiCad board)
At the start: 2 copper layers, 100 x 100 mm, 7 parts, among them J1 Conn_01x35_Pin, U1 SN74CBT3244PW

Commit message: Add files via upload
New version with better footprint and ground isolation.
Parts:
- U1: footprint Package_SO:TSSOP-20_4.4x6.5mm_P0.65mm -> Package_SO:SOIC-20W_7.5x12.8mm_P1.27mm
- moved C1 23.3 mm to (150.0, 98.0), turned to -90 degrees
- moved U1 22.5 mm to (141.8, 103.3)
Connections:
- JAud1 pad 1: Net-(JAud1-IN1-Pad1) -> Net-(U1-1A1)
- JAud1 pad 3: Net-(U1-1A1) -> Net-(JAud1-IN1-Pad3)
- JAud1 pad 4: GND -> Net-(JAud1-GND)
- RVR2 pad 1: Net-(JAud1-IN1-Pad1) -> Net-(JAud1-IN1-Pad3)
- U1 pad 12: unconnected-(U1-1B4-Pad12) -> GND
- U1 pad 14: unconnected-(U1-1B3-Pad14) -> GND
- U1 pad 16: unconnected-(U1-1B2-Pad16) -> /Comp
- U1 pad 4: unconnected-(U1-1A2-Pad4) -> Net-(U1-1A1)
- U1 pad 6: unconnected-(U1-1A3-Pad6) -> Net-(JAud1-GND)
- U1 pad 8: unconnected-(U1-1A4-Pad8) -> Net-(JAud1-GND)
Routing:
- net Net-(JAud1-GND): track 0.00 -> 72.7 mm, vias 0 -> 1
- net Net-(JAud1-IN1-Pad1): track 69.9 -> 0.00 mm
- net Net-(JAud1-IN1-Pad3): track 0.00 -> 41.9 mm
- net Net-(JP1-A): track 74.0 -> 94.4 mm
- net /Comp: track 43.1 -> 62.2 mm, vias 1 -> 0
- net GND: track 177.0 -> 161.0 mm
- net /ACTIVE: track 65.1 -> 49.3 mm
- net /R_AUD: track 52.1 -> 36.9 mm
- net /L_AUD: track 48.6 -> 36.9 mm
- net +5V: track 65.4 -> 55.5 mm
- net Net-(U1-1A1): track 38.0 -> 45.6 mm, vias 0 -> 1
- net Net-(JAud1-IN2): track 70.8 -> 64.2 mm
- net Net-(JP1-B): track 91.5 -> 85.2 mm
