File: AVSwitch-VGA/AVSwitch-VGA.kicad_pcb (KiCad board)
At the start: 2 copper layers, 100 x 100 mm, 9 parts, among them J1 Conn_01x35_Pin, J2 DE15_Receptacle_HighDensity_M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, U1 SN74CBT3244PW

Commit message: Add files via upload
New version with better footprint and ground isolation.
Parts:
- U1: footprint Package_SO:TSSOP-20_4.4x6.5mm_P0.65mm -> Package_SO:SOIC-20W_7.5x12.8mm_P1.27mm
- moved C1 43.4 mm to (157.0, 93.5), turned to 90 degrees
- moved U1 26.9 mm to (152.7, 104.2), turned to 0 degrees
Connections:
- J2 pad 0: GND -> Net-(JLaud1-Ext)
- J2 pad 1: Net-(U1-1A1) -> Net-(U1-2A1)
- J2 pad 10: GND -> Net-(JLaud1-Ext)
- J2 pad 13: Net-(U1-1A4) -> Net-(U1-1A3)
- J2 pad 14: Net-(U1-2A1) -> Net-(U1-1A4)
- J2 pad 2: Net-(U1-1A3) -> Net-(U1-2A2)
- J2 pad 3: Net-(U1-1A2) -> Net-(U1-2A3)
- J2 pad 5: GND -> Net-(JLaud1-Ext)
- J2 pad 6: GND -> Net-(JLaud1-Ext)
- J2 pad 7: GND -> Net-(JLaud1-Ext)
- J2 pad 8: GND -> Net-(JLaud1-Ext)
- JLaud1 pad 2: GND -> Net-(JLaud1-Ext)
- JRaud1 pad 2: GND -> Net-(JLaud1-Ext)
- U1 pad 12: /V_H -> /V_V
- U1 pad 13: Net-(JP1-B) -> Net-(U1-2A2)
- U1 pad 14: /V_B -> /V_H
- U1 pad 15: unconnected-(U1-2A3-Pad15) -> Net-(U1-2A3)
- U1 pad 16: /V_G -> /L_AUD
- U1 pad 17: Net-(JP1-A) -> Net-(JLaud1-Ext)
- U1 pad 18: /V_R -> /R_AUD
- U1 pad 2: Net-(U1-1A1) -> Net-(JP1-A)
- U1 pad 3: /R_AUD -> GND
- U1 pad 4: Net-(U1-1A2) -> Net-(JP1-B)
- U1 pad 5: unconnected-(U1-2B3-Pad5) -> /V_B
- U1 pad 7: /L_AUD -> /V_G
- U1 pad 9: /V_V -> /V_R
Routing:
- net Net-(JLaud1-Ext): track 0.00 -> 122.7 mm
- net Net-(U1-2A3): track 0.00 -> 47.6 mm
- net Net-(U1-1A1): track 47.0 -> 0.00 mm
- net Net-(U1-1A2): track 45.4 -> 0.00 mm, vias 2 -> 0
- net Net-(U1-2A2): track 0.00 -> 42.8 mm
- net /ACTIVE: track 77.9 -> 107.2 mm
- net GND: track 235.2 -> 210.1 mm
- net Net-(U1-2A1): track 64.7 -> 39.6 mm, vias 1 -> 0
- net /V_H: track 33.7 -> 52.8 mm, vias 0 -> 1
- net Net-(JP1-A): track 82.3 -> 101.0 mm, vias 1 -> 0
- net /V_R: track 28.4 -> 43.6 mm
- net /V_V: track 40.7 -> 54.2 mm, vias 0 -> 1
- net /V_G: track 30.1 -> 42.6 mm
- net +5V: track 88.4 -> 76.1 mm, vias 2 -> 0
- net Net-(U1-1A4): track 61.2 -> 50.3 mm, vias 2 -> 1
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